File: Projects/tractor/schematic/relay_changed/v2.4/bundle/tractor_2v4.brd (EAGLE design)
At the start: 66.5 x 45.5 mm, 80 parts, among them IC1 PIC16F1824, IC2 33063A, K2 RL703, Q1 IRLML2402, Q2 IRLML2402, Q3 IRLML2402, T1 BC547

Commit message: 2V4 release
Parts:
- removed T1: BC547, transistor-neu-to92:TO92
- added Q4: 2N2222, transistor-npn:TO18
- K2: value RL703 -> RL3531RL3; device relay:RL703 -> relay:RL3531
- R12: device eagle-ltspice:R3216 -> eagle-ltspice:R2010
- R8: value 470 -> 220
- moved R8 14.6 mm to (43.7, 7.70), turned to 90 degrees
- moved D4 6.11 mm to (55.3, 9.23), turned to 90 degrees
- moved D11 5.85 mm to (30.0, 8.60), turned to 270 degrees
- moved D2 4.66 mm to (41.5, 5.70), turned to 90 degrees
- moved C16 4.25 mm to (35.6, 7.30)
- moved R23 3.62 mm to (55.0, 19.2), turned to 270 degrees
- moved R12 2.70 mm to (7.20, 28.5)
- moved C1 1.71 mm to (47.5, 31.5)
- moved R6 1.70 mm to (48.6, 28.0)
- moved K2 1.66 mm to (49.5, 33.4), flipped to the top, turned to 90 degrees
- moved D1 1.65 mm to (49.4, 41.2)
- moved Q1 1.65 mm to (47.6, 34.6)
- moved R11 1.62 mm to (52.0, 5.79)
- moved C5 1.50 mm to (4.10, 17.5)
- moved R5 1.30 mm to (46.8, 27.9)
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Connections:
- removed net BUZZ_4: BUZ.1, D4.K, R11.1
- removed net N$14: D2.K, T1.2
- removed net N$90: R11.2, T1.3
- new net N$13: Q4.3, R11.2
- new net N$16: BUZ.1, D4.A, R11.1
- new net N$37: 0V.1, B1.AC2
- net 12V_8: now also D4.K, K2.NC
- net GND: now also Q4.1; no longer D4.A, T1.1
- net N$1: now also Q4.2, R8.2; no longer 0V.1, B1.AC2, K2.NO
- net N$5: now also K2.L2; no longer K2.1
- net N$7: now also D2.K; no longer D2.A
- net N$88: now also D2.A; no longer R8.2
- net VDD: now also K2.L1; no longer K2.2
Routing:
- net N$1: track 39.9 -> 3.54 mm
- net 12V_8: track 44.4 -> 75.8 mm, vias 0 -> 2
- net N$37: track 0.00 -> 31.3 mm
- net N$88: track 31.2 -> 42.2 mm
- net BUZZ_4: track 10.3 -> 0.00 mm
- net N$16: track 0.00 -> 7.51 mm
- net N$90: track 7.40 -> 0.00 mm
- net GND: track 253.6 -> 246.8 mm
- net N$7: track 8.35 -> 2.86 mm
- net N$82: track 35.9 -> 40.0 mm
- net N$14: track 3.54 -> 0.00 mm
- net N$13: track 0.00 -> 2.55 mm
- net N$76: track 25.8 -> 23.6 mm
- net N$33: track 15.6 -> 13.6 mm
- net R_3: track 9.02 -> 11.1 mm
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
Commit message: schematic changes
Parts:
- renumbered PAD_3 to SOL
Changed lines of the file:
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@@
 <layer number="14" name="Route14" color="1" fill="6" visible="no" active="no"/>
 <layer number="15" name="Route15" color="4" fill="6" visible="no" active="no"/>
-<layer number="16" name="Bottom" color="1" fill="1" visible="yes" active="yes"/>
+<layer number="16" name="Bottom" color="1" fill="1" visible="no" active="yes"/>
 <layer number="17" name="Pads" color="2" fill="1" visible="yes" active="yes"/>
 <layer number="18" name="Vias" color="2" fill="1" visible="yes" active="yes"/>
@@
 <layer number="20" name="Dimension" color="15" fill="1" visible="yes" active="yes"/>
 <layer number="21" name="tPlace" color="7" fill="1" visible="yes" active="yes"/>
-<layer number="22" name="bPlace" color="7" fill="1" visible="yes" active="yes"/>
+<layer number="22" name="bPlace" color="7" fill="1" visible="no" active="yes"/>
 <layer number="23" name="tOrigins" color="15" fill="1" visible="yes" active="yes"/>
-<layer number="24" name="bOrigins" color="15" fill="1" visible="yes" active="yes"/>
+<layer number="24" name="bOrigins" color="15" fill="1" visible="no" active="yes"/>
 <layer number="25" name="tNames" color="7" fill="1" visible="yes" active="yes"/>
-<layer number="26" name="bNames" color="7" fill="1" visible="yes" active="yes"/>
+<layer number="26" name="bNames" color="7" fill="1" visible="no" active="yes"/>
 <layer number="27" name="tValues" color="7" fill="1" visible="no" active="yes"/>
 <layer number="28" name="bValues" color="7" fill="1" visible="no" active="yes"/>
@@
 <layer number="38" name="bTest" color="7" fill="1" visible="no" active="yes"/>
 <layer number="39" name="tKeepout" color="4" fill="11" visible="yes" active="yes"/>
-<layer number="40" name="bKeepout" color="1" fill="11" visible="yes" active="yes"/>
+<layer number="40" name="bKeepout" color="1" fill="11" visible="no" active="yes"/>
 <layer number="41" name="tRestrict" color="4" fill="10" visible="yes" active="yes"/>
-<layer number="42" name="bRestrict" color="1" fill="10" visible="yes" active="yes"/>
+<layer number="42" name="bRestrict" color="1" fill="10" visible="no" active="yes"/>
 <layer number="43" name="vRestrict" color="2" fill="10" visible="no" active="yes"/>
 <layer number="44" name="Drills" color="7" fill="1" visible="no" active="yes"/>
@@
 <layer number="49" name="Reference" color="7" fill="1" visible="no" active="yes"/>
 <layer number="51" name="tDocu" color="7" fill="1" visible="yes" active="yes"/>
-<layer number="52" name="bDocu" color="7" fill="1" visible="yes" active="yes"/>
+<layer number="52" name="bDocu" color="7" fill="1" visible="no" active="yes"/>
 <layer number="90" name="Modules" color="5" fill="1" visible="no" active="no"/>
 <layer number="91" name="Nets" color="2" fill="1" visible="no" active="no"/>
@@
 <attribute name="VALUE" x="63.6407" y="39.63065625" size="0.0254" layer="27" rot="R180"/>
 </element>
-<element name="PAD_3" library="wirepad" package="2,54/1,1" value="" x="63.965525" y="33.872403125" rot="R180">
+<element name="SOL" library="wirepad" package="2,54/1,1" value="" x="63.965525" y="33.872403125" rot="R180">
 <attribute name="VALUE" x="63.965525" y="32.872403125" size="0.0254" layer="27" rot="R180"/>
 </element>
@@
 </signal>
 <signal name="R_3">
-<contactref element="PAD_3" pad="1"/>
+<contactref element="SOL" pad="1"/>
 <contactref element="K2" pad="C1"/>
 <wire x1="63.965525" y1="33.872403125" x2="60.727596875" y2="33.872403125" width="2.54" layer="1"/>
