File: Projects/tractor/schematic/relay_changed/v2.4/bundle/tractor_2v4.sch (EAGLE design)
At the start: 80 parts, among them IC1 PIC16F1824, IC2 33063A, K2 RL703, Q1 IRLML2402, Q2 IRLML2402, Q3 IRLML2402, T1 BC547

Commit message: 2V4 release
Parts:
- removed T1: BC547, transistor-neu-to92:BC547
- added Q4: 2N2222, transistor-npn:2N2222
- K2: value RL703 -> RL3531RL3; device relay:RL703 -> relay:RL3531RL3
- R12: device eagle-ltspice:RR3216 -> eagle-ltspice:RR2010
- R8: value 470 -> 220
Connections:
- removed net BUZZ_4: BUZ.P, D4.C, R11.1
- removed net N$14: D2.C, T1.B
- removed net N$90: R11.2, T1.C
- new net N$13: Q4.C, R11.2
- new net N$16: BUZ.P, D4.A, R11.1
- new net N$37: 0V.P, B1.AC2
- net 12V_8: now also D4.C, K2.NC
- net GND: now also Q4.E; no longer D4.A, T1.E
- net N$1: now also Q4.B, R8.2; no longer 0V.P, B1.AC2, K2.NO
- net N$7: now also D2.C; no longer D2.A
- net N$88: now also D2.A; no longer R8.2
Other:
- note added: "03-Jan-2019"
- note added: "Version:- 2.4"
- note removed: "24-Oct-2018"
- note removed: "Version:- 2.3"
- moved on the sheet: +12V, 0V, B1, BUZ, C1, C10, C11, C12, C13, C15, C16, C17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

Commit message: schematic changes
Parts:
- renumbered PAD_3 to SOL
Other:
- note added: "Version:- 2.4.1"
- note removed: "Version:- 2.4"
Changed lines of the file:
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@@
 <part name="0V" library="wirepad" deviceset="2,54/1,1" device="" value="0V"/>
 <part name="+12V" library="wirepad" deviceset="2,54/1,1" device="" value="+12V"/>
-<part name="PAD_3" library="wirepad" deviceset="2,54/1,1" device=""/>
+<part name="SOL" library="wirepad" deviceset="2,54/1,1" device=""/>
 <part name="ENG_9" library="wirepad" deviceset="2,54/1,1" device=""/>
 <part name="PTO" library="wirepad" deviceset="2,54/1,1" device=""/>
@@
 <wire x1="157.48" y1="0" x2="190.5" y2="0" width="0.1524" layer="94"/>
 <text x="161.13799375" y="9.538525" size="1.27" layer="94" align="top-center">Name:-</text>
-<text x="163.36895" y="2.00005" size="1.27" layer="94" align="top-center">Version:- 2.4</text>
+<text x="163.86895" y="2.00005" size="1.27" layer="94" align="top-center">Version:- 2.4.1</text>
 <text x="160.657003125" y="6.91876875" size="1.27" layer="94" align="top-center">Date:-</text>
 <text x="169.101040625" y="9.431596875" size="1.27" layer="94" align="top-center">ECU - Driver</text>
@@
 <attribute name="VALUE" x="3.937" y="141.478" size="1.778" layer="96"/>
 </instance>
-<instance part="PAD_3" gate="1" x="22.86" y="124.46" rot="MR270">
-<attribute name="NAME" x="21.0058" y="125.603" size="1.778" layer="95" rot="MR270"/>
+<instance part="SOL" gate="1" x="22.86" y="124.46" rot="MR270">
 <attribute name="VALUE" x="26.162" y="125.603" size="1.778" layer="96" rot="MR270"/>
 </instance>
@@
 <segment>
 <wire x1="22.86" y1="116.84" x2="22.86" y2="121.92" width="0.1524" layer="91"/>
-<pinref part="PAD_3" gate="1" pin="P"/>
+<pinref part="SOL" gate="1" pin="P"/>
 <junction x="22.86" y="121.92"/>
 <pinref part="K2" gate="G$1" pin="C1"/>
@@
 </sheet>
 </sheets>
-<errors>
-</errors>
 </schematic>
 </drawing>
