File: Projects/tractor_ECU/Hardware/ECU_1v0/ECU_1v0.brd (EAGLE design)
At the start: 95.7 x 81.2 mm, 142 parts, among them IC2 33063A, IC4 PIC16F1718, Q10 IRFR5305, Q11 IRFR5305, Q5 IRLML2402, Q6 IRLML2402, Q7 IRLML2402, Q8 IRLML2402, Q9 IRLML2402

Commit message: v2.5 bug fix
Parts:
- removed +12V: +12V, wirepad:2,54/1,1
- removed 0V: 0V, wirepad:2,54/1,1
- removed BUZZER, ENG_CTL_GOV, ENG_ST_UP, IGN_SW, MID_PTO, NEUTRAL_IND, N_W_SW, OPC(NC), OPC(NO), PARK_BRAKE_IND, PTO_LW, PTO_SAFE_ST, P_B_SW, ST_COIL_RL, ST_MOTOR: (no value), wirepad:2,54/1,1
- removed C26, C27, C28: 470uf, resistor:C050-075X075
- removed C29, C30, C31, C32, C33, C34, C35: 1nf, eagle-ltspice:C0603
- removed D13, D14, D15, D16, D17, D18, D19, D20, D21, D22, D23, D24, D25, D26, D27, D28: Fm4007, diode:SMA-DO214AC
- removed FERITE: FB MH1608HM151-T, resistor:R0603
- removed IC4: PIC16F1718, microchip:SO28W
- removed PR20: 50, resistor:WSC2515
- removed Q10, Q11: IRFR5305, transistor-power:D-PAK_TO252AA
- removed Q8, Q9: IRLML2402, transistor-power:MICRO3
- removed R32, R33, R71, R72, R73, R74, R75, R76, R77: 1.5k, eagle-ltspice:R0603
- removed R34, R35, R36, R37, R38, R59, R60, R61, R62, R63, R64, R65, R66, R67, R68, R69, R70: 10k, eagle-ltspice:R0603
- added BUZ, ENG_CTRL_GOV, NTRL_IND, PAD12, PAD13, PAD14, PAD15, PAD5, PAD6, PAD7, PAD8, PAD9, PARK_BRK_IND, STRT_MOT, STRT_REL_COIL: (no value), wirepad:2,54/1,1
- added C1: 10uf, eagle-ltspice:C0603
- added C10: 0.01uf, eagle-ltspice:C0603
- added C11, C13, C16, C18, C2: 470uf, resistor:C050-075X075
- added C17: 0.01uF, eagle-ltspice:C0603
- added C6: 1nf, eagle-ltspice:C0603
- added C9: 100uf, rcl:C025-025X050
- added D1, D10, D11, D12, D2, D3, D4, D8, D9: Fm4007, diode:SMA-DO214AC
- added D7: 1N5819, diode:SMA-DO214AC
- added GND, RX, TX: (no value), wirepad:1,6/0,8
- added IC1: PIC16F1718, microchip:SO28W
- added PAD1: +12V, wirepad:2,54/1,1
- added PAD2: 0V, wirepad:2,54/1,1
- added Q1, Q2, Q3, Q4: IRLML2402, transistor-power:MICRO3
- added R1: 10K, eagle-ltspice:R0603
- added R11: FB MH1608HM151-T, resistor:R0603
- added R14, R16, R20, R3, R6, R8: 1.5k, eagle-ltspice:R0603
- added R15, R17, R19, R2, R5, R7, R9: 4.5k, eagle-ltspice:R0603
- added R21: 3.6k, eagle-ltspice:R0603
- added R22: 1.2k, eagle-ltspice:R0603
- added R23: 330m, eagle-ltspice:R2010
- added R4: S20K17, varistor:S14K17
- C12: value 4nf -> 100nf; device rcl:C050-045X075 -> eagle-ltspice:C0603
- C14: value 10uf -> 470pf
- C15: value 470uf -> 220uf; device resistor:C050-075X075 -> rcl:C025-025X050
- C19: value 100nf -> 1nf
- C24, C25: value 470uf -> 1nf; device resistor:C050-075X075 -> eagle-ltspice:C0603
- C3: value 0.01uf -> 1nf
- C4: value 0.01uF -> 4nf; device eagle-ltspice:C0603 -> rcl:C050-045X075
- C5: value 220uf -> 1nf; device rcl:C025-025X050 -> eagle-ltspice:C0603
- C7: value 470pf -> 1nf
- C8: value 100uf -> 470uf; device rcl:C025-025X050 -> resistor:C050-075X075
- D6: value 1N5819 -> Fm4007
- Q6, Q7: value IRLML2402 -> IRFR5305; device transistor-power:MICRO3 -> transistor-power:D-PAK_TO252AA
- R10: value S20K17 -> 1.5k; device varistor:S14K17 -> eagle-ltspice:R0603
- R12: value 330m -> 50; device eagle-ltspice:R2010 -> resistor:WSC2515
- R13: value 3.6k -> 4.5k
- R18: value 1.2k -> 1.5k
- R24: value 10K -> 10k
- R25, R26, R27, R28, R29, R30: value 1.5k -> 10k
- R31: value 1.5k -> 4.5k
- R39, R57, R58: value 10k -> 1.5k
- R48, R49, R50, R51, R52, R53: value 4.5k -> 10k
- R54, R55, R56: value 4.5k -> 1.5k
- moved R39 1105.0 mm to (75.2, 47.6), turned to 180 degrees
- moved R40 1081.7 mm to (71.6, 20.3), flipped to the bottom, turned to 180 degrees
- moved CLR 1066.3 mm to (16.9, 55.1), turned to 90 degrees
- moved Q6 1062.6 mm to (74.0, 32.6), turned to 90 degrees
- moved Q5 1062.0 mm to (77.2, 32.2), flipped to the bottom, turned to 90 degrees
- moved VCC 1057.7 mm to (16.8, 62.5), turned to 90 degrees
- moved Q7 1055.2 mm to (73.9, 24.3), turned to 90 degrees
- moved CLK 1039.3 mm to (16.9, 60.0), turned to 90 degrees
- moved DAT 1020.9 mm to (16.9, 57.6), turned to 90 degrees
- moved PTO_SOL 802.0 mm to (86.4, 32.8)
- moved R57 637.0 mm to (80.8, 42.6), flipped to the bottom, turned to 270 degrees
- moved R58 630.9 mm to (80.4, 32.3), flipped to the bottom, turned to 270 degrees
- moved R56 627.7 mm to (80.8, 37.4), flipped to the bottom, turned to 270 degrees
- moved R55 613.6 mm to (80.4, 27.3), flipped to the bottom, turned to 270 degrees
- moved R54 604.1 mm to (81.7, 21.4), flipped to the bottom, turned to 180 degrees
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Connections:
- removed net N$109: Q11.4, R77.1
- removed net N$110: Q10.4, R76.1
- removed net N$117: D27.A, NEUTRAL_IND.1, R74.2
- removed net N$118: BUZZER.1, D26.A, R75.2
- removed net N$119: D25.A, R72.2, ST_MOTOR.1
- removed net N$120: D22.A, R71.2, ST_COIL_RL.1
- removed net N$121: D23.A, ENG_CTL_GOV.1, R76.2
- removed net N$122: D24.A, PTO_SOL.1, R77.2
- removed net N$65: IC4.4, OK1.12, R50.1
- removed net N$70: IC4.10, OK2.10, R55.1
- removed net N$71: IC4.11, OK3.16, R56.1
- removed net N$73: IC4.13, R46.1
- removed net N$75: IC4.14, R45.1
- removed net N$77: IC4.15, R44.1
- removed net N$79: IC4.16, R43.1
- removed net N$80: IC4.17, R42.1
- removed net N$81: IC4.18, R41.1
- new net 12V_R: F1.2, Q6.4, Q7.4, R11.1, R55.2, R56.2, R57.2, R58.2
- new net N$1: IC1.4, R30.1
- new net N$13: IC1.14, OK1.10, R9.1
- new net N$16: IC1.24, R27.1
- new net N$17: IC1.22, R25.1
- new net N$24: Q4.2, STRT_MOT.1
- new net N$25: Q5.2, STRT_REL_COIL.1
- new net N$26: PTO_SOL.1, Q6.3
- new net N$27: ENG_CTRL_GOV.1, Q7.3
- new net N$28: IC1.18, RX.1
- new net N$3: IC1.21, R24.1
- new net N$30: IC1.17, TX.1
- new net N$5: PARK_BRK_IND.1, Q2.2
- new net N$6: IC1.10, OK2.10, R19.1
- new net N$7: IC1.11, OK1.16, R2.1
- new net N$8: IC1.23, R26.1
- new net N$9: IC1.13, OK1.12, R7.1
- net 12V_8: now also D12.K, PAD1.1; no longer +12V.1, D22.K, D23.K, D24.K, D25.K, D26.K, D27.K, D28.K
- net GND: now also C1.1, C10.1, C11.2, C12.1, C13.2, C16.2, C17.1, C18.2, C2.2, C24.1, C25.1, C4.2, C5.1, C6.1, C9.2, D1.A, D10.A, D3.A, D7.A, D8.A, GND.1, IC1.19, IC1.8, Q1.2, R22.2, R4.1, R41.2, R43.2, R45.2, R47.2, R49.2, R51.2, R53.2; no longer C12.2, C24.2, C25.2, C26.2, C27.2, C28.2, C29.1, C30.1, C31.1, C32.1, C33.1, C34.1, C35.1, C4.1, C5.2, D14.A, D16.A, D18.A, D20.A, D6.A, IC4.19, IC4.8, Q10.3, Q11.3, Q5.2, Q6.2, Q7.2, Q8.2, Q9.2, R10.1, R18.2, R34.2, R35.2, R36.2, R37.2, R38.2, R39.2, R40.2, R58.2, R60.2, R62.2, R64.2, R66.2, R68.2, R70.2
- net N$100: now also OK3.11, R44.1, R45.1; no longer OK4.13, R36.1, R61.1, R62.1
- net N$101: now also C22.2, Q4.1, R46.2; no longer C32.2, Q5.1, R63.2
- net N$102: now also OK3.13, R46.1, R47.1; no longer OK4.15, R37.1, R63.1, R64.1
- net N$103: now also C23.2, Q5.1, R48.2; no longer C33.2, Q9.1, R65.2
- net N$104: now also R48.1, R49.1; no longer R38.1, R65.1, R66.1
- net N$105: now also C24.2, Q6.1, R50.2; no longer C34.2, Q10.1, R67.2
- net N$106: now also OK4.13, R50.1, R51.1; no longer OK3.11, R39.1, R67.1, R68.1
- net N$107: now also C25.2, Q7.1, R52.2; no longer C35.2, Q11.1, R69.2
- net N$108: now also OK4.15, R52.1, R53.1; no longer OK3.13, R40.1, R69.1, R70.1
- net N$111: now also Q1.3, R54.1; no longer Q8.3, R73.1
- net N$112: now also Q2.3, R55.1; no longer Q7.3, R74.1
- net N$113: now also Q3.3, R56.1; no longer Q6.3, R75.1
- net N$114: now also Q4.3, R57.1; no longer Q5.3, R72.1
- net N$115: now also Q5.3, R58.1; no longer Q9.3, R71.1
- net N$116: now also D12.A, NTRL_IND.1, R54.2; no longer D28.A, PARK_BRAKE_IND.1, R73.2
- net N$123: now also IC1.28; no longer IC4.28
- net N$124: now also IC1.27; no longer IC4.27
- net N$14: now also C1.2, IC1.1, R1.2; no longer C14.2, IC4.1, R24.2
- net N$15: now also R11.2, R12.1; no longer FERITE.2, PR20.1
- net N$18: now also R23.1; no longer R12.1
- net N$19: now also C14.2; no longer C7.2
- net N$20: now also BUZ.1, Q3.2; no longer F1.2, FERITE.1
- net N$21: now also L1.1; no longer L2.1
- net N$22: now also D7.K, L2.2; no longer D6.K, L1.2
- net N$23: now also R21.2, R22.1; no longer R13.2, R18.1
- net N$29: now also C2.1, C4.1, L1.2, R4.2; no longer C12.1, C15.1, L2.2, R10.2
- net N$35: now also C3.2, PAD5.1, R3.2; no longer C20.2, OPC(NO).1, R25.2
- net N$37: now also PAD2.1; no longer 0V.1
- net N$38: now also C5.2, PAD6.1, R6.2; no longer C21.2, OPC(NC).1, R26.2
- net N$39: now also C6.2, PAD7.1, R8.2; no longer C22.2, P_B_SW.1, R27.2
- net N$40: now also C7.2, PAD8.1, R10.2; no longer C23.2, N_W_SW.1, R28.2
- net N$41: now also C8.1, D1.K, R14.2; no longer C24.1, D5.K, R29.2
- net N$42: now also D2.K, R14.1; no longer D13.K, R29.1
- net N$43: now also D2.A, PAD9.1; no longer D13.A, IGN_SW.1
- net N$44: now also C11.1, D3.K, R16.2; no longer C25.1, D14.K, R30.2
- net N$45: now also D4.K, R16.1; no longer D15.K, R30.1
- net N$46: now also D4.A, PAD12.1; no longer D15.A, ENG_ST_UP.1
- net N$47: now also C13.1, D5.K, R18.2; no longer C26.1, D16.K, R31.2
- net N$48: now also D6.K, R18.1; no longer D17.K, R31.1
- net N$49: now also D6.A, PAD13.1; no longer D17.A, PTO_SAFE_ST.1
- net N$50: now also C16.1, D8.K, R20.2; no longer C27.1, D18.K, R32.2
- net N$51: now also D9.K, R20.1; no longer D19.K, R32.1
- net N$52: now also D9.A, PAD14.1; no longer D19.A, MID_PTO.1
- net N$53: now also C18.1, D10.K, R39.2; no longer C28.1, D20.K, R33.2
- net N$54: now also D11.K, R39.1; no longer D21.K, R33.1
- net N$55: now also D11.A, PAD15.1; no longer D21.A, PTO_LW.1
- net N$56: now also R24.2; no longer R41.2
- net N$57: now also R25.2; no longer R42.2
- net N$58: now also R26.2; no longer R43.2
- net N$59: now also R27.2; no longer R44.2
- net N$60: now also R28.2; no longer R45.2
- net N$61: now also R29.2; no longer R46.2
- net N$62: now also R30.2; no longer R47.2
- net N$63: now also IC1.2, R28.1; no longer IC4.2, OK1.16, R48.1
- net N$64: now also IC1.3, R29.1; no longer IC4.3, OK1.14, R49.1
- net N$66: now also IC1.5, OK3.16, R31.1; no longer IC4.5, OK1.10, R51.1
- net N$67: now also IC1.6, R13.1; no longer IC4.6, R52.1
- net N$68: now also IC1.7, R15.1; no longer IC4.7, R53.1
- net N$69: now also IC1.9, R17.1; no longer IC4.9, R54.1
- net N$83: now also IC1.12, OK1.14, R5.1; no longer IC4.12, R47.1
- net N$86: now also C19.2, Q1.1, R40.2; no longer C29.2, Q8.1, R57.2
- net N$96: now also C20.2, Q2.1, R42.2; no longer C30.2, Q7.1, R59.2
- net N$97: now also OK4.11, R40.1, R41.1; no longer OK4.9, R34.1, R57.1, R58.1
- net N$98: now also OK4.9, R42.1, R43.1; no longer OK4.11, R35.1, R59.1, R60.1
- net N$99: now also C21.2, Q3.1, R44.2; no longer C31.2, Q6.1, R61.2
- net VCC: now also C12.2, C15.1, C17.2, IC1.20, L2.1, OK3.10, OK3.12, OK3.14, OK4.10, OK4.12, OK4.14, OK4.16, R1.1, R13.2, R15.2, R17.2, R19.2, R2.2, R21.1, R31.2, R5.2, R7.2, R9.2; no longer C19.2, C4.2, C5.1, IC4.20, L1.1, R13.1, R24.1, R48.2, R49.2, R50.2, R51.2, R52.2, R53.2, R54.2, R55.2, R56.2
- net VDD: now also C10.2, C9.1, R10.1, R23.2, R3.1, R6.1, R8.1; no longer C3.2, C8.1, OK3.10, OK3.12, OK3.14, OK4.10, OK4.12, OK4.14, OK4.16, PR20.2, R25.1, R26.1, R27.1, R28.1
Routing:
- net GND: track 79.3 -> 536.8 mm, vias 0 -> 7
- net VCC: track 16.1 -> 224.5 mm, vias 0 -> 11
- net VDD: track 38.1 -> 152.8 mm, vias 1 -> 4
- net 12V_R: track 0.00 -> 90.5 mm, vias 0 -> 4
- net N$53: track 0.00 -> 41.8 mm
- net N$16: track 0.00 -> 41.8 mm, vias 0 -> 1
- net N$8: track 0.00 -> 41.3 mm, vias 0 -> 1
- net N$17: track 0.00 -> 40.5 mm, vias 0 -> 1
- net N$3: track 0.00 -> 39.6 mm, vias 0 -> 1
- net N$13: track 0.00 -> 36.6 mm
- net N$9: track 0.00 -> 35.9 mm
- net N$7: track 0.00 -> 35.6 mm
- net N$83: track 0.00 -> 35.3 mm
- net N$66: track 0.00 -> 33.1 mm, vias 0 -> 2
- net N$41: track 0.00 -> 32.7 mm
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Other:
- board size 95.7 x 81.2 mm -> 84.7 x 77.4 mm
