File: Projects/tractor_ECU/Hardware/ECU_1v0/ECU_1v0.sch (EAGLE design)
At the start: 142 parts, among them IC2 33063A, IC4 PIC16F1718, Q10 IRFR5305, Q11 IRFR5305, Q5 IRLML2402, Q6 IRLML2402, Q7 IRLML2402, Q8 IRLML2402, Q9 IRLML2402

Commit message: v2.5 bug fix
Parts:
- removed BUZZER, ENG_CTL_GOV, ENG_ST_UP, IGN_SW, MID_PTO, NEUTRAL_IND, N_W_SW, OPC(NC), OPC(NO), PARK_BRAKE_IND, PTO_LW, PTO_SAFE_ST, P_B_SW, ST_COIL_RL, ST_MOTOR: (no value), wirepad:2,54/1,1
- removed C26, C27, C28: 470uf, resistor:C-US050-075X075
- removed C29, C30, C31, C32, C33, C34, C35: 1nf, eagle-ltspice:CC0603
- removed D13, D14, D15, D16, D17, D18, D19, D20, D21, D22, D23, D24, D25, D26, D27, D28: Fm4007, diode:GF1
- removed IC4: PIC16F1718, microchip:PIC16F1516/18SO
- removed PR20: 50, resistor:R-US_WSC2515
- removed Q10, Q11: IRFR5305, transistor-power:IRFR5305
- removed Q8, Q9: IRLML2402, transistor-power:IRLML5203
- removed R32, R33, R71, R72, R73, R74, R75, R76, R77: 1.5k, eagle-ltspice:RR0603
- removed R34, R35, R36, R37, R38, R59, R60, R61, R62, R63, R64, R65, R66, R67, R68, R69, R70: 10k, eagle-ltspice:RR0603
- added BUZ, ENG_CTRL_GOV, NTRL_IND, PAD12, PAD13, PAD14, PAD15, PAD5, PAD6, PAD7, PAD8, PAD9, PARK_BRK_IND, STRT_MOT, STRT_REL_COIL: (no value), wirepad:2,54/1,1
- added C1: 10uf, eagle-ltspice:CC0603
- added C10: 0.01uf, eagle-ltspice:CC0603
- added C11, C13, C16, C18, C2: 470uf, resistor:C-US050-075X075
- added C17: 0.01uF, eagle-ltspice:CC0603
- added C6: 1nf, eagle-ltspice:CC0603
- added C9: 100uf, rcl:C-US025-025X050
- added D1, D10, D11, D12, D2, D3, D4, D8, D9: Fm4007, diode:GF1
- added D7: 1N5819, diode:GF1
- added GND, RX, TX: (no value), wirepad:1,6/0,8
- added IC1: PIC16F1718, microchip:PIC16F1516/18SO
- added Q1, Q2, Q3, Q4: IRLML2402, transistor-power:IRLML5203
- added R1: 10K, eagle-ltspice:RR0603
- added R14, R16, R20, R3, R6, R8: 1.5k, eagle-ltspice:RR0603
- added R15, R17, R19, R2, R5, R7, R9: 4.5k, eagle-ltspice:RR0603
- added R21: 3.6k, eagle-ltspice:RR0603
- added R22: 1.2k, eagle-ltspice:RR0603
- added R23: 330m, eagle-ltspice:RR2010
- added R4: S20K17, varistor:S14K17
- C12: value 4nf -> 100nf; device rcl:C-US050-045X075 -> eagle-ltspice:CC0603
- C14: value 10uf -> 470pf
- C15: value 470uf -> 220uf; device resistor:C-US050-075X075 -> rcl:C-US025-025X050
- C19: value 100nf -> 1nf
- C24, C25: value 470uf -> 1nf; device resistor:C-US050-075X075 -> eagle-ltspice:CC0603
- C3: value 0.01uf -> 1nf
- C4: value 0.01uF -> 4nf; device eagle-ltspice:CC0603 -> rcl:C-US050-045X075
- C5: value 220uf -> 1nf; device rcl:C-US025-025X050 -> eagle-ltspice:CC0603
- C7: value 470pf -> 1nf
- C8: value 100uf -> 470uf; device rcl:C-US025-025X050 -> resistor:C-US050-075X075
- D6: value 1N5819 -> Fm4007
- Q6, Q7: value IRLML2402 -> IRFR5305; device transistor-power:IRLML5203 -> transistor-power:IRFR5305
- R10: value S20K17 -> 1.5k; device varistor:S14K17 -> eagle-ltspice:RR0603
- R12: value 330m -> 50; device eagle-ltspice:RR2010 -> resistor:R-US_WSC2515
- R13: value 3.6k -> 4.5k
- R18: value 1.2k -> 1.5k
- R24: value 10K -> 10k
- R25, R26, R27, R28, R29, R30: value 1.5k -> 10k
- R31: value 1.5k -> 4.5k
- R39, R57, R58: value 10k -> 1.5k
- R48, R49, R50, R51, R52, R53: value 4.5k -> 10k
- R54, R55, R56: value 4.5k -> 1.5k
- renumbered +12V to PAD1, 0V to PAD2, FERITE to R11
Connections:
- removed net N$109: Q11.D, R77.1
- removed net N$110: Q10.D, R76.1
- removed net N$117: D27.A, NEUTRAL_IND.P, R74.2
- removed net N$118: BUZZER.P, D26.A, R75.2
- removed net N$119: D25.A, R72.2, ST_MOTOR.P
- removed net N$120: D22.A, R71.2, ST_COIL_RL.P
- removed net N$121: D23.A, ENG_CTL_GOV.P, R76.2
- removed net N$122: D24.A, PTO_SOL.P, R77.2
- removed net N$65: IC4.AN2/RA2, OK1C.COL, R50.1
- removed net N$70: IC4.CLKOUT/OSC2/RA6, OK2D.COL, R55.1
- removed net N$71: IC4.T1CKI/SOSCO/RC0, OK3A.COL, R56.1
- removed net N$73: IC4.CCP1/AN14/RC2, R46.1
- removed net N$75: IC4.SCL/SCK/AN15/RC3, R45.1
- removed net N$77: IC4.RC4/AN16/SDI/SDA, R44.1
- removed net N$79: IC4.RC5/AN17/SDO, R43.1
- removed net N$80: IC4.RC6/AN18/TX/CK, R42.1
- removed net N$81: IC4.RC7/AN19/RX/DT, R41.1
- new net 12V_R: F1.4, Q6.D, Q7.D, R11.1, R55.2, R56.2, R57.2, R58.2
- new net N$1: IC1.AN2/RA2, R30.1
- new net N$13: IC1.SCL/SCK/AN15/RC3, OK1D.COL, R9.1
- new net N$16: IC1.RB3/AN9/CCP2, R27.1
- new net N$17: IC1.RB1/AN10, R25.1
- new net N$24: Q4.S, STRT_MOT.P
- new net N$25: Q5.S, STRT_REL_COIL.P
- new net N$26: PTO_SOL.P, Q6.S
- new net N$27: ENG_CTRL_GOV.P, Q7.S
- new net N$28: IC1.RC7/AN19/RX/DT, RX.P
- new net N$3: IC1.RB0/AN12/INT, R24.1
- new net N$30: IC1.RC6/AN18/TX/CK, TX.P
- new net N$5: PARK_BRK_IND.P, Q2.S
- new net N$6: IC1.CLKOUT/OSC2/RA6, OK2D.COL, R19.1
- new net N$7: IC1.T1CKI/SOSCO/RC0, OK1A.COL, R2.1
- new net N$8: IC1.RB2/AN8, R26.1
- new net N$9: IC1.CCP1/AN14/RC2, OK1C.COL, R7.1
- net 12V_8: now also D12.C; no longer D22.C, D23.C, D24.C, D25.C, D26.C, D27.C, D28.C
- net GND: now also C1.1, C10.1, C11.2, C12.1, C13.2, C16.2, C17.1, C18.2, C2.2, C24.1, C25.1, C4.2, C5.1, C6.1, C9.2, D1.A, D10.A, D3.A, D7.A, D8.A, GND.P, IC1.VSS, IC1.VSS@1, Q1.S, R22.2, R4.1, R41.2, R43.2, R45.2, R47.2, R49.2, R51.2, R53.2; no longer C12.2, C24.2, C25.2, C26.2, C27.2, C28.2, C29.1, C30.1, C31.1, C32.1, C33.1, C34.1, C35.1, C4.1, C5.2, D14.A, D16.A, D18.A, D20.A, D6.A, IC4.VSS, IC4.VSS@1, Q10.S, Q11.S, Q5.S, Q6.S, Q7.S, Q8.S, Q9.S, R10.1, R18.2, R34.2, R35.2, R36.2, R37.2, R38.2, R39.2, R40.2, R58.2, R60.2, R62.2, R64.2, R66.2, R68.2, R70.2
- net N$100: now also OK3C.EMIT, R44.1, R45.1; no longer OK4B.EMIT, R36.1, R61.1, R62.1
- net N$101: now also C22.2, Q4.G, R46.2; no longer C32.2, Q5.G, R63.2
- net N$102: now also OK3B.EMIT, R46.1, R47.1; no longer OK4A.EMIT, R37.1, R63.1, R64.1
- net N$103: now also C23.2, Q5.G, R48.2; no longer C33.2, Q9.G, R65.2
- net N$104: now also R48.1, R49.1; no longer R38.1, R65.1, R66.1
- net N$105: now also C24.2, Q6.G, R50.2; no longer C34.2, Q10.G, R67.2
- net N$106: now also OK4B.EMIT, R50.1, R51.1; no longer OK3C.EMIT, R39.1, R67.1, R68.1
- net N$107: now also C25.2, Q7.G, R52.2; no longer C35.2, Q11.G, R69.2
- net N$108: now also OK4A.EMIT, R52.1, R53.1; no longer OK3B.EMIT, R40.1, R69.1, R70.1
- net N$111: now also Q1.D, R54.1; no longer Q8.D, R73.1
- net N$112: now also Q2.D, R55.1; no longer Q7.D, R74.1
- net N$113: now also Q3.D, R56.1; no longer Q6.D, R75.1
- net N$114: now also Q4.D, R57.1; no longer Q5.D, R72.1
- net N$115: now also Q5.D, R58.1; no longer Q9.D, R71.1
- net N$116: now also D12.A, NTRL_IND.P, R54.2; no longer D28.A, PARK_BRAKE_IND.P, R73.2
- net N$123: now also IC1.RB7/ICSPDAT/ICDDAT; no longer IC4.RB7/ICSPDAT/ICDDAT
- net N$124: now also IC1.RB6/ICSPCLK/ICDCLK; no longer IC4.RB6/ICSPCLK/ICDCLK
- net N$14: now also C1.2, IC1.VPP/!MCLR!/RE3, R1.2; no longer C14.2, IC4.VPP/!MCLR!/RE3, R24.2
- net N$15: now also R12.1; no longer PR20.1
- net N$18: now also R23.1; no longer R12.1
- net N$19: now also C14.2; no longer C7.2
- net N$20: now also BUZ.P, Q3.S; no longer F1.4, R11.1
- net N$21: now also L1.1; no longer L2.1
- net N$22: now also D7.C, L2.2; no longer D6.C, L1.2
- net N$23: now also R21.2, R22.1; no longer R13.2, R18.1
- net N$29: now also C2.1, C4.1, L1.2, R4.2; no longer C12.1, C15.1, L2.2, R10.2
- net N$35: now also C3.2, PAD5.P, R3.2; no longer C20.2, OPC(NO).P, R25.2
- net N$38: now also C5.2, PAD6.P, R6.2; no longer C21.2, OPC(NC).P, R26.2
- net N$39: now also C6.2, PAD7.P, R8.2; no longer C22.2, P_B_SW.P, R27.2
- net N$40: now also C7.2, PAD8.P, R10.2; no longer C23.2, N_W_SW.P, R28.2
- net N$41: now also C8.1, D1.C, R14.2; no longer C24.1, D5.C, R29.2
- net N$42: now also D2.C, R14.1; no longer D13.C, R29.1
- net N$43: now also D2.A, PAD9.P; no longer D13.A, IGN_SW.P
- net N$44: now also C11.1, D3.C, R16.2; no longer C25.1, D14.C, R30.2
- net N$45: now also D4.C, R16.1; no longer D15.C, R30.1
- net N$46: now also D4.A, PAD12.P; no longer D15.A, ENG_ST_UP.P
- net N$47: now also C13.1, D5.C, R18.2; no longer C26.1, D16.C, R31.2
- net N$48: now also D6.C, R18.1; no longer D17.C, R31.1
- net N$49: now also D6.A, PAD13.P; no longer D17.A, PTO_SAFE_ST.P
- net N$50: now also C16.1, D8.C, R20.2; no longer C27.1, D18.C, R32.2
- net N$51: now also D9.C, R20.1; no longer D19.C, R32.1
- net N$52: now also D9.A, PAD14.P; no longer D19.A, MID_PTO.P
- net N$53: now also C18.1, D10.C, R39.2; no longer C28.1, D20.C, R33.2
- net N$54: now also D11.C, R39.1; no longer D21.C, R33.1
- net N$55: now also D11.A, PAD15.P; no longer D21.A, PTO_LW.P
- net N$56: now also R24.2; no longer R41.2
- net N$57: now also R25.2; no longer R42.2
- net N$58: now also R26.2; no longer R43.2
- net N$59: now also R27.2; no longer R44.2
- net N$60: now also R28.2; no longer R45.2
- net N$61: now also R29.2; no longer R46.2
- net N$62: now also R30.2; no longer R47.2
- net N$63: now also IC1.!SS!/AN0/RA0, R28.1; no longer IC4.!SS!/AN0/RA0, OK1A.COL, R48.1
- net N$64: now also IC1.AN1/RA1, R29.1; no longer IC4.AN1/RA1, OK1B.COL, R49.1
- net N$66: now also IC1.VREF+/AN3/RA3, OK3A.COL, R31.1; no longer IC4.VREF+/AN3/RA3, OK1D.COL, R51.1
- net N$67: now also IC1.T0CKI/RA4, R13.1; no longer IC4.T0CKI/RA4, R52.1
- net N$68: now also IC1.VCAP/!SS!/AN4/RA5, R15.1; no longer IC4.VCAP/!SS!/AN4/RA5, R53.1
- net N$69: now also IC1.CLKIN/OSC1/RA7, R17.1; no longer IC4.CLKIN/OSC1/RA7, R54.1
- net N$83: now also IC1.CCP2/SOSCI/RC1, OK1B.COL, R5.1; no longer IC4.CCP2/SOSCI/RC1, R47.1
- net N$86: now also C19.2, Q1.G, R40.2; no longer C29.2, Q8.G, R57.2
- net N$96: now also C20.2, Q2.G, R42.2; no longer C30.2, Q7.G, R59.2
- net N$97: now also OK4C.EMIT, R40.1, R41.1; no longer OK4D.EMIT, R34.1, R57.1, R58.1
- net N$98: now also OK4D.EMIT, R42.1, R43.1; no longer OK4C.EMIT, R35.1, R59.1, R60.1
- net N$99: now also C21.2, Q3.G, R44.2; no longer C31.2, Q6.G, R61.2
- net VCC: now also C12.2, C15.1, C17.2, IC1.VDD, L2.1, OK3B.COL, OK3C.COL, OK3D.COL, OK4A.COL, OK4B.COL, OK4C.COL, OK4D.COL, R1.1, R13.2, R15.2, R17.2, R19.2, R2.2, R21.1, R31.2, R5.2, R7.2, R9.2; no longer C19.2, C4.2, C5.1, IC4.VDD, L1.1, R13.1, R24.1, R48.2, R49.2, R50.2, R51.2, R52.2, R53.2, R54.2, R55.2, R56.2
- net VDD: now also C10.2, C9.1, R10.1, R23.2, R3.1, R6.1, R8.1; no longer C3.2, C8.1, OK3B.COL, OK3C.COL, OK3D.COL, OK4A.COL, OK4B.COL, OK4C.COL, OK4D.COL, PR20.2, R25.1, R26.1, R27.1, R28.1
Other:
- moved on the sheet: C12, C14, C15, C19, C20, C21, C22, C23, C24, C25, C3, C4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
